Commit message: Add files via upload

File: back_arm.xacro (robot description, xacro)
@@ -1,8 +1,8 @@
 <?xml version="1.0"?>
 <robot xmlns:xacro="http://www.ros.org/wiki/xacro" name="my_robot">
-<xacro:macro name="arm" params="prefix radius length reflect">
+<xacro:macro name="back_arm" params="prefix radius length reflect">
     <!-- rpy (roll pitch yaw) describes rotation in radians -->
     <!-- xyz describes translation in meters -->
-    <link name="${prefix}_arm">
+    <link name="${prefix}_back_arm">
         <visual>
             <origin rpy="0 1.57 1.57" xyz="0 0 0"/> <!-- set the origin to 0 to recenter the link to the child_frame -->
@@ -23,17 +23,17 @@
         </inertial>
     </link>
-    <joint name="base_to_${prefix}_arm" type="continuous">
+    <joint name="base_to_${prefix}_back_arm" type="continuous">
         <axis xyz="0 1 0"/>
         <parent link="base_link"/>
-        <child link="${prefix}_arm"/>
-        <origin rpy="0 0 0" xyz="0.7 ${reflect*0.5} 0"/> <!-- move the child_frame with respect to parent_frame -->
+        <child link="${prefix}_back_arm"/>
+        <origin rpy="0 0 0" xyz="-0.9 ${reflect*0.6} 0"/> <!-- move the child_frame with respect to parent_frame -->
         <limit effort="30" velocity="2.0"/>
     </joint>
-    <transmission name="${prefix}_arm_transmission">
+    <transmission name="${prefix}_back_arm_transmission">
         <type>transmission_interface/SimpleTransmission</type>
         <actuator name="$${prefix}_motor">
             <mechanicalReduction>1</mechanicalReduction>
         </actuator>
-        <joint name="base_to_${prefix}_arm">
+        <joint name="base_to_${prefix}_back_arm">
             <hardwareInterface>hardware_interface/VelocityJointInterface</hardwareInterface>
         </joint>

File: head.xacro (robot description, xacro)
@@ -25,5 +25,5 @@
         <parent link="base_link"/>
         <child link="head_link"/>
-        <origin rpy="0 0 0" xyz="0 0 .5"/> <!-- moves the child_frame with respect to parent_frame -->
+        <origin rpy="0 0 0" xyz="0 0 .145"/> <!-- moves the child_frame with respect to parent_frame -->
         <limit effort="30" velocity="1.0"/>
     </joint>

File: main.xacro (robot description, xacro)
@@ -3,13 +3,14 @@
     <xacro:include filename="$(find tutorial)/urdf/arm.xacro" />
     <xacro:include filename="$(find tutorial)/urdf/head.xacro" />
+    <xacro:include filename="$(find tutorial)/urdf/back_arm.xacro" />
     <link name="base_link">
         <visual>
             <geometry>
-                <box size="1 1 1"/>
+                <box size="2 1.5 0.3"/>
             </geometry>
         </visual>
         <collision>
             <geometry>
-                <box size="1 1 1"/>
+                <box size="2 1.5 0.3"/>
             </geometry>
         </collision>
@@ -19,6 +20,8 @@
         </inertial>
     </link>
-    <xacro:arm prefix="right" length="1.2" radius=".2" reflect="1" />
-    <xacro:arm prefix="left" length="1.2" radius=".2" reflect="-1" />
+    <xacro:arm prefix="right" length=".1" radius="0.5" reflect="1" />
+    <xacro:arm prefix="left" length=".1" radius="0.5" reflect="-1" />
+    <xacro:back_arm prefix="right" length=".1" radius="0.7" reflect="1" />
+    <xacro:back_arm prefix="left" length=".1" radius="0.7" reflect="-1" />
     <xacro:head />
     <!-- Add ROS plugin so we can interact with our robot -->
